File: board.brd (EAGLE design)
At the start: 100 x 80 mm, 32 parts, among them IC1 7805T, J1 350428-1

Commit message: Atualizando espessura das linhas e reorganizando
Parts:
- moved C2 72.9 mm to (20.3, 52.1)
- moved C4 44.5 mm to (14.0, 61.0)
- moved C7 35.9 mm to (20.3, 40.6), turned to 180 degrees
- moved IC1 30.6 mm to (40.6, 43.2), turned to 180 degrees
- moved C3 28.0 mm to (39.4, 61.0)
- moved R2 25.0 mm to (74.9, 54.6), turned to 90 degrees
- moved C11 18.2 mm to (54.6, 59.7), turned to 90 degrees
- moved C8 17.8 mm to (25.4, 61.0), turned to 180 degrees
- moved 7905 12.7 mm to (6.35, 43.2)
- moved C12 5.39 mm to (72.4, 63.5)
- moved C10 1.27 mm to (83.8, 59.7)

Commit message: Linhas automáticas
Parts:
- moved C1 17.8 mm to (77.5, 22.9)
- moved C6 16.1 mm to (69.8, 44.5)
- moved IC2 14.0 mm to (80.0, 35.6), turned to 270 degrees
- moved C9 5.24 mm to (83.8, 50.8)
- moved C11 4.02 mm to (55.9, 63.5)
- moved ADJ 3.81 mm to (94.0, 72.4)
- moved C5 2.84 mm to (83.8, 55.9)
- moved C10 2.84 mm to (82.5, 62.2)
Routing:
- net GND: track 0.00 -> 273.8 mm
- net N$6: track 0.00 -> 133.8 mm
- net N$10: track 0.00 -> 128.2 mm
- net N$4: track 0.00 -> 75.6 mm
- net N$11: track 0.00 -> 74.4 mm
- net N$9: track 0.00 -> 63.2 mm
- net N$8: track 0.00 -> 39.4 mm
- net N$13: track 0.00 -> 36.9 mm
- net N$2: track 0.00 -> 33.9 mm
- net N$12: track 0.00 -> 26.9 mm
- net N$1: track 0.00 -> 24.4 mm
- net N$3: track 0.00 -> 21.8 mm
- net N$5: track 0.00 -> 17.1 mm
- net N$7: track 0.00 -> 15.9 mm
- net N$14: track 0.00 -> 14.6 mm
